Commit message: main

File: midterm/xacro/model/sensor/lidar/lidar.xacro (robot description, xacro)
@@ -2,5 +2,5 @@
 <robot xmlns:xacro="http://www.ros.org/wiki/xacro">
     <xacro:macro name="lidar">
-        <link name="lidar">
+        <link name="lindar">
             <inertial>
                 <origin xyz="-0.00829409957033964 -6.93889390390723E-18 0.010701142222791" rpy="0 0 0" />
@@ -27,9 +27,9 @@
             <origin xyz="0.108 0 0.042" rpy="0 0 0" />
             <parent link="base_link" />
-            <child link="lidar" />
+            <child link="lindar" />
             <axis xyz="0 0 0" />
             <dynamics damping="0.1" friction="0.1" />
         </joint>
-    <gazebo reference="lidar">
+    <gazebo reference="lindar">
       <sensor type="ray" name="lidar_sensor">
         <pose>0 0 0 0 0 0</pose>

File: midterm/xacro/model/wheel/wheel.xacro (robot description, xacro)
@@ -69,5 +69,5 @@
         <origin xyz="0 0 0" rpy="0 0 0" />
         <geometry>
-          <mesh filename="package://midterm/urdf/meshes/Left_backward_wheel.STL" />
+          <mesh filename="package://midterm/urdf/meshes/Right_backward_wheel.STL" />
         </geometry>
         <material name="">
@@ -78,5 +78,5 @@
         <origin xyz="0 0 0" rpy="0 0 0" />
         <geometry>
-          <mesh filename="package://midterm/urdf/meshes/Left_backward_wheel.STL" />
+          <mesh filename="package://midterm/urdf/meshes/Right_backward_wheel.STL" />
         </geometry>
       </collision>
@@ -98,5 +98,5 @@
         <origin xyz="0 0 0" rpy="0 0 0" />
         <geometry>
-          <mesh filename="package://midterm/urdf/meshes/Right_backward_wheel.STL" />
+          <mesh filename="package://midterm/urdf/meshes/Left_backward_wheel.STL" />
         </geometry>
         <material name="">
@@ -107,5 +107,5 @@
         <origin xyz="0 0 0" rpy="0 0 0" />
         <geometry>
-          <mesh filename="package://midterm/urdf/meshes/Right_backward_wheel.STL" />
+          <mesh filename="package://midterm/urdf/meshes/Left_backward_wheel.STL" />
         </geometry>
       </collision>
